Commit message: fls link

File: alpha_rise_description/urdf/base.urdf.xacro (robot description, xacro)
@@ -69,4 +69,10 @@
         <child link="ping360_link_sf"/>
     </joint>
+    <link name="fls_link_sf"/>
+    <joint name="fls_sf_joint" type="fixed">
+        <origin xyz="0.4 -0.2 0.0" rpy="1.57 0.0 -1.57"/>
+        <parent link="base_link"/>
+        <child link="fls_link_sf"/>
+    </joint>
     <!-- thrusters -->
     <link name="surge_thruster_link"/>

Commit message: wakefield test config

File: alpha_rise_description/urdf/base.urdf.xacro (robot description, xacro)
@@ -69,4 +69,16 @@
         <child link="ping360_link_sf"/>
     </joint>
+    <link name="fls_link"/>
+    <joint name="fls_link_joint" type="fixed">
+        <origin xyz="0.4 -0.2 0.0" rpy="1.57 0.0 -1.57"/>
+        <parent link="base_link"/>
+        <child link="fls_link"/>
+    </joint>
+    <link name="fls_link_sf"/>
+    <joint name="fls_link_joint_sf" type="fixed">
+        <origin xyz="0.4 -0.2 0.0" rpy="1.57 0.0 -1.57"/>
+        <parent link="base_link"/>
+        <child link="fls_link_sf"/>
+    </joint>
     <!-- thrusters -->
     <link name="surge_thruster_link"/>

Commit message: fix: tf for IMU & FLS

File: alpha_rise_description/urdf/base.urdf.xacro (robot description, xacro)
@@ -23,5 +23,5 @@
     <link name="imu"/>
     <joint name="imu_joint" type="fixed">
-        <origin xyz="-0.2 -0.0 0.0" rpy="0 0.0 0.0"/>
+        <origin xyz="-0.18 -0.0 0.15" rpy="0 0.0 0.0"/>
         <parent link="base_link"/>
         <child link="imu"/>
@@ -71,5 +71,5 @@
     <link name="fls_link"/>
     <joint name="fls_link_joint" type="fixed">
-        <origin xyz="0.4 -0.2 0.0" rpy="1.57 0.0 -1.57"/>
+        <origin xyz="-0.3 -0.2 0.0" rpy="1.57 0.0 -1.57"/>
         <parent link="base_link"/>
         <child link="fls_link"/>
@@ -77,11 +77,5 @@
     <link name="fls_link_sf"/>
     <joint name="fls_link_joint_sf" type="fixed">
-        <origin xyz="0.4 -0.2 0.0" rpy="1.57 0.0 -1.57"/>
-        <parent link="base_link"/>
-        <child link="fls_link_sf"/>
-    </joint>
-    <link name="fls_link_sf"/>
-    <joint name="fls_sf_joint" type="fixed">
-        <origin xyz="0.4 -0.2 0.0" rpy="1.57 0.0 -1.57"/>
+        <origin xyz="-0.3 -0.2 0.0" rpy="1.57 0.0 -1.57"/>
         <parent link="base_link"/>
         <child link="fls_link_sf"/>

Commit message: fix: ping360 & pressure link adjustments

File: alpha_rise_description/urdf/base.urdf.xacro (robot description, xacro)
@@ -53,5 +53,5 @@
     <link name="pressure"/>
     <joint name="pressure_joint" type="fixed">
-        <origin xyz="0.3 0.0 0.05" rpy="3.1415926 0.0 0.0"/>
+        <origin xyz="0.17 -0.07 0.05" rpy="3.1415926 0.0 0.0"/>
         <parent link="base_link"/>
         <child link="pressure"/>
@@ -59,5 +59,5 @@
     <link name="ping360_link"/>
     <joint name="ping360_joint" type="fixed">
-        <origin xyz="0.63 0.0 -0.085" rpy="0.0 0.0 3.1415926"/>
+        <origin xyz="0.63 0.0 -0.11" rpy="0.0 0.0 3.1415926"/>
         <parent link="base_link"/>
         <child link="ping360_link"/>
@@ -65,5 +65,5 @@
     <link name="ping360_link_sf"/>
     <joint name="ping360_sf_joint" type="fixed">
-        <origin xyz="0.63 0.0 -0.085" rpy="3.14 0.0 0.0"/>
+        <origin xyz="0.63 0.0 -0.11" rpy="3.14 0.0 0.0"/>
         <parent link="base_link"/>
         <child link="ping360_link_sf"/>
