Commit message: feat: tested for simulation

File: alpha_rise_description/urdf/base.urdf (robot description, URDF)
Before this commit: robot alpha_rise, 17 links, 16 joints
Joints:
- joint gps_joint: origin xyz=0.05 0.0 0.32 rpy=0.0 0.0 0.0 -> xyz=0.05 0.0 0.32 rpy=3.1415926 0.0 0.0
- joint imu__sf_joint: origin xyz=0.0 0.0 0.0 rpy=3.1415926 0.0 0.0 -> xyz=0.0 0.0 0.0 rpy=0.0 0.0 0.0
- joint pressure_joint: origin xyz=0.17 -0.07 0.05 rpy=3.1415926 0.0 0.0 -> xyz=0.3 0.0 0.05 rpy=3.1415926 0.0 0.0

Commit message: change: z of surge thruster set to 0.0. added xyz_flag for surge thruster

File: alpha_rise_description/urdf/base.urdf (robot description, URDF)
Before this commit: robot alpha_rise, 17 links, 16 joints
Joints:
- joint surge_thruster_joint: origin xyz=-0.77 0.0 0.02 rpy=0.0 0.0 0.0 -> xyz=-0.77 0.0 0.0 rpy=0.0 0.0 0.0

Commit message: change: dvl tf

File: alpha_rise_description/urdf/base.urdf (robot description, URDF)
Before this commit: robot alpha_rise, 17 links, 16 joints
Joints:
- joint dvl_joint: origin xyz=0.51 0.0 -0.1 rpy=3.1415926 0.0 0.0 -> xyz=-0.18 0.0 -0.1 rpy=3.1415926 0.0 0.0

Commit message: feat: added rtk launch, yaml. fused rtk heading to microstrain. changed localization cov params

File: alpha_rise_description/urdf/base.urdf (robot description, URDF)
Before this commit: robot alpha_rise, 17 links, 16 joints
Links:
- removed link gps
- added link unicore_gps
Joints:
- removed joint gps_joint
- added joint unicore_gps_joint: type fixed, parent base_link, child unicore_gps, origin xyz=-0.5875 0.0 0.2 rpy=3.1415926 0.0 0.0
- joint dvl_joint: origin xyz=-0.18 0.0 -0.1 rpy=3.1415926 0.0 0.0 -> xyz=-0.18 0.0 -0.127 rpy=3.1415926 0.0 0.0
- joint imu_joint: origin xyz=-0.18 -0.0 0.15 rpy=0 0.0 0.0 -> xyz=-0.18 -0.0 -0.15 rpy=0 0.0 0.0

Commit message: fix: urdf

File: alpha_rise_description/urdf/base.urdf (robot description, URDF)
Before this commit: robot alpha_rise, 17 links, 16 joints
Joints:
- joint base_link: origin xyz=0.72 0.0 0.0 rpy=0.0 0.0 0.0 -> xyz=0.76 0.0 0.0 rpy=0.0 0.0 0.0
- joint cg_joint: origin xyz=-0.06 0.0 0.0 rpy=3.1415926 0.0 0.0 -> xyz=-0.0 0.0 0.0 rpy=3.1415926 0.0 0.0
- joint dvl_joint: origin xyz=-0.18 0.0 -0.127 rpy=3.1415926 0.0 0.0 -> xyz=-0.04 0.0 -0.17 rpy=3.1415926 0.0 0.0
- joint fls_link_joint: origin xyz=-0.3 -0.2 0.0 rpy=1.57 0.0 -1.57 -> xyz=-0.26 -0.2 0.0 rpy=1.57 0.0 -1.57
- joint heave_bow_thruster_joint: origin xyz=0.387 0.0 0.0 rpy=0.0 -1.57079632679 0.0 -> xyz=0.42 0.0 0.0 rpy=0.0 -1.57079632679 0.0
- joint imu_joint: origin xyz=-0.18 -0.0 -0.15 rpy=0 0.0 0.0 -> xyz=-0.04 -0.0 -0.15 rpy=0 0.0 0.0
- joint ping360_joint: origin xyz=0.63 0.0 -0.11 rpy=0.0 0.0 3.1415926 -> xyz=0.70 0.0 -0.11 rpy=0.0 0.0 3.1415926
- joint surge_thruster_joint: origin xyz=-0.77 0.0 0.0 rpy=0.0 0.0 0.0 -> xyz=-0.74 0.0 0.0 rpy=0.0 0.0 0.0
- joint unicore_gps_joint: origin xyz=-0.5875 0.0 0.2 rpy=3.1415926 0.0 0.0 -> xyz=-0.5 0.0 0.2 rpy=3.1415926 0.0 0.0

Commit message: corrected tf for FLS

File: alpha_rise_description/urdf/base.urdf (robot description, URDF)
Before this commit: robot alpha_rise, 17 links, 16 joints
Joints:
- joint fls_link_joint: origin xyz=-0.26 -0.2 0.0 rpy=1.57 0.0 -1.57 -> xyz=-0.26 -0.13 0.0 rpy=1.57 0.0 -1.57

Commit message: mbes tf & launch files

File: alpha_rise_description/urdf/base.urdf (robot description, URDF)
Before this commit: robot alpha_rise, 17 links, 16 joints
Links:
- added link mbes_link
Joints:
- added joint mbes_joint: type fixed, parent base_link, child mbes_link, origin xyz=0.74 -0.10 -0.0 rpy=0.0 1.57 -0.7854
- joint ping360_joint: origin xyz=0.70 0.0 -0.11 rpy=0.0 0.0 3.1415926 -> xyz=0.74 0.0 -0.11 rpy=0.0 0.0 3.1415926

Commit message: fix: gps link 0 roll

File: alpha_rise_description/urdf/base.urdf (robot description, URDF)
Before this commit: robot alpha_rise, 18 links, 17 joints
Joints:
- joint unicore_gps_joint: origin xyz=-0.5 0.0 0.2 rpy=3.1415926 0.0 0.0 -> xyz=-0.5 0.0 0.2 rpy=0.0 0.0 0.0

Commit message: fix: unicore inverted

File: alpha_rise_description/urdf/base.urdf (robot description, URDF)
Before this commit: robot alpha_rise, 18 links, 17 joints
Joints:
- joint unicore_gps_joint: origin xyz=-0.5 0.0 0.2 rpy=0.0 0.0 0.0 -> xyz=-0.5 0.0 0.2 rpy=3.1415926 0.0 0.0

Commit message: params, added mbes_sf link, autonomy launch

File: alpha_rise_description/urdf/base.urdf (robot description, URDF)
Before this commit: robot alpha_rise, 18 links, 17 joints
Links:
- added link mbes_link_sf
Joints:
- added joint mbes_sf_joint: type fixed, parent base_link, child mbes_link_sf, origin xyz=0.74 -0.10 -0.0 rpy=3.1415926 -0.0 -0.785

Commit message: wall following params and fls urdf

File: alpha_rise_description/urdf/base.urdf (robot description, URDF)
Before this commit: robot alpha_rise, 19 links, 18 joints
Links:
- removed link fls_link
- added link fls
Joints:
- joint fls_link_joint: child fls_link -> fls

Commit message: tfs

File: alpha_rise_description/urdf/base.urdf (robot description, URDF)
Before this commit: robot alpha_rise, 19 links, 18 joints
Joints:
- joint heave_stern_thruster_joint: origin xyz=-0.4 0.0 0.0 rpy=0.0 -1.57079632679 0.0 -> xyz=-0.37 0.0 0.0 rpy=0.0 -1.57079632679 0.0
- joint ping360_joint: origin xyz=0.74 0.0 -0.11 rpy=0.0 0.0 3.1415926 -> xyz=0.7 0.0 -0.15 rpy=0.0 0.0 3.1415926
- joint pressure_joint: origin xyz=0.3 0.0 0.05 rpy=3.1415926 0.0 0.0 -> xyz=0.13 0.0 0.05 rpy=3.1415926 0.0 0.0
- joint surge_thruster_joint: origin xyz=-0.74 0.0 0.0 rpy=0.0 0.0 0.0 -> xyz=-0.78 0.0 0.0 rpy=0.0 0.0 0.0
- joint sway_bow_thruster_joint: origin xyz=0.51 0.0 0.0 rpy=0.0 0.0 1.57079632679 -> xyz=0.53 0.0 0.0 rpy=0.0 0.0 1.57079632679
- joint unicore_gps_joint: origin xyz=-0.5 0.0 0.2 rpy=3.1415926 0.0 0.0 -> xyz=-0.46 0.0 0.2 rpy=3.1415926 0.0 0.0
